File: hardware/STM32F446VE-Module/STM32F446VE-Module.kicad_pcb (KiCad board)
At the start: 4 copper layers, 65 x 45 mm, 88 parts, among them J1 USB_C_Receptacle_USB2.0, J2 Conn_ARM_SWD_TagConnect_TC2030, J3 Micro_SD_Card_Det_Hirose_DM3AT, J4 DF40C-60DP-0.4V_51_, J5 DF40C-60DP-0.4V_51_, J6 BM02B-GHS-TBT(LF)(SN), J7 BM04B-GHS-TBT(LF)(SN), J8 BM04B-GHS-TBT(LF)(SN), SW1 SW_Push, SW2 SW_DIP_x02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

Commit message: Prepare for fab
Other:
- rule pad_to_mask_clearance: 0.038 -> 0
Changed lines of the file:
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@@
       (dielectric_constraints no)
     )
-    (pad_to_mask_clearance 0.038)
-    (solder_mask_min_width 0.1)
-    (aux_axis_origin 104 54)
+    (pad_to_mask_clearance 0)
+    (aux_axis_origin 104 99)
+    (grid_origin 104 99)
     (pcbplotparams
       (layerselection 0x00010fc_ffffffff)
@@
       (viasonmask false)
       (mode 1)
-      (useauxorigin false)
+      (useauxorigin true)
       (hpglpennumber 1)
       (hpglpenspeed 20)
@@
       (outputformat 1)
       (mirror false)
-      (drillshape 1)
+      (drillshape 0)
       (scaleselection 1)
-      (outputdirectory "")
+      (outputdirectory "output/")
     )
   )
@@
     (fp_line (start 1.6 0.8) (end 1.6 -0.8)
       (stroke (width 0.1) (type solid)) (layer "F.Fab"))
-    (pad "1" smd roundrect (at -1.4375 0 90) (size 1.575 1.35) (layers "F.Cu" "F.Paste" "F.Mask") (roundrect_rratio 0.185185)
+    (pad "1" smd roundrect (at -1.4375 0 90) (size 1.575 1.35) (layers "F.Cu" "F.Paste" "F.Mask") (roundrect_rratio 0.1851851852)
       (net 4 "+3.3V") (pintype "passive"))
-    (pad "2" smd roundrect (at 1.4375 0 90) (size 1.575 1.35) (layers "F.Cu" "F.Paste" "F.Mask") (roundrect_rratio 0.185185)
+    (pad "2" smd roundrect (at 1.4375 0 90) (size 1.575 1.35) (layers "F.Cu" "F.Paste" "F.Mask") (roundrect_rratio 0.1851851852)
       (net 2 "GND") (pintype "passive"))
     (model "${KICAD6_3DMODEL_DIR}/Capacitor_Tantalum_SMD.3dshapes/CP_EIA-3216-18_Kemet-A.wrl"
@@
     (pad "26" smd rect (at -1 1.355) (size 0.23 0.66) (layers "B.Cu" "B.Paste" "B.Mask")
       (net 104 "/PE9") (pinfunction "26") (pintype "passive"))
-    (pad "27" smd rect locked (at -0.6 -1.355) (size 0.23 0.66) (layers "B.Cu" "B.Paste" "B.Mask")
+    (pad "27" smd rect (at -0.6 -1.355) (size 0.23 0.66) (layers "B.Cu" "B.Paste" "B.Mask")
       (net 22 "/CAN-") (pinfunction "27") (pintype "passive"))
     (pad "28" smd rect (at -0.6 1.355) (size 0.23 0.66) (layers "B.Cu" "B.Paste" "B.Mask")
@@
     (polygon
       (pts
-        (xy 125.2598 86.0552)
+        (xy 125.2598 85.5)
         (xy 126.733 84.988)
         (xy 128.9682 84.988)

Commit message: send for fab
Parts:
- R19: footprint Capacitor_SMD:C_0603_1608Metric_Pad1.08x0.95mm_HandSolder -> Resistor_SMD:R_0603_1608Metric_Pad0.98x0.95mm_HandSolder
Connections:
- J4 pad 26: /PE9 -> /CAN+
- J4 pad 27: /CAN- -> /PE9
- J4 pad 28: /PE10 -> /CAN-
- J4 pad 29: /CAN+ -> /PE10
- J4 pad 30: /PE11 -> unconnected-(J4-Pad30)
- J4 pad 31: unconnected-(J4-Pad31) -> /PE11
- J4 pad 32: /PE12 -> unconnected-(J4-Pad32)
- J4 pad 33: unconnected-(J4-Pad33) -> /PE12
- J4 pad 34: /PE13 -> unconnected-(J4-Pad34)
- J4 pad 35: unconnected-(J4-Pad35) -> /PE13
- J4 pad 36: /PE14 -> unconnected-(J4-Pad36)
- J4 pad 37: unconnected-(J4-Pad37) -> /PE14
- J4 pad 39: unconnected-(J4-Pad39) -> /PE15
- J4 pad 41: unconnected-(J4-Pad41) -> /PB10
- J4 pad 42: /PE15 -> unconnected-(J4-Pad42)
- J4 pad 44: /PB10 -> unconnected-(J4-Pad44)
Routing:
- net /PE12: track 40.2 -> 28.6 mm, vias 3 -> 1
- net /PE10: track 37.7 -> 26.7 mm, vias 3 -> 1
- net /PE14: track 44.8 -> 34.0 mm
- net /PE11: track 37.5 -> 27.5 mm, vias 3 -> 1
- net /PE15: track 44.0 -> 34.4 mm
- net /PE13: track 41.4 -> 32.0 mm
- net /PE9: track 34.8 -> 25.7 mm, vias 3 -> 1
- net /PB10: track 43.8 -> 35.2 mm
- net /CAN+: track 63.0 -> 61.7 mm
- net VBUS: vias 4 -> 5
- net +VDC: vias 6 -> 7
