File: hardware/STM32F446VE-Module/STM32F446VE-Module.kicad_sch (KiCad schematic)
At the start: 88 parts, among them J1 USB_C_Receptacle_USB2.0, J2 Conn_ARM_SWD_TagConnect_TC2030, J3 Micro_SD_Card_Det_Hirose_DM3AT, J4 DF40C-60DP-0.4V_51_, J5 DF40C-60DP-0.4V_51_, J6 BM02B-GHS-TBT(LF)(SN), J7 BM04B-GHS-TBT(LF)(SN), J8 BM04B-GHS-TBT(LF)(SN), SW1 SW_Push, SW2 SW_DIP_x02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

Commit message: Prepare for fab
Parts:
- D7: JLCPCB C441887 -> C72038
- TP1, TP10, TP2, TP3, TP4, TP5, TP6, TP7, TP8, TP9: now left out of the parts list
Other:
- note added: "Conn A"
- note added: "Conn B"

Commit message: send for fab
Parts:
- J1: JLCPCB (none) -> C3020560
- R19: footprint Capacitor_SMD:C_0603_1608Metric_Pad1.08x0.95mm_HandSolder -> Resistor_SMD:R_0603_1608Metric_Pad0.98x0.95mm_HandSolder
- SW1: JLCPCB (none) -> C5504987
- U5: JLCPCB (none) -> C91929
Connections:
- net CAN+: now also J4.26; no longer J4.29
- net CAN-: now also J4.28; no longer J4.27
- net PB10: now also J4.41; no longer J4.44
- net PE10: now also J4.29; no longer J4.28
- net PE11: now also J4.31; no longer J4.30
- net PE12: now also J4.33; no longer J4.32
- net PE13: now also J4.35; no longer J4.34
- net PE14: now also J4.37; no longer J4.36
- net PE15: now also J4.39; no longer J4.42
- net PE9: now also J4.27; no longer J4.26
Changed lines of the file:
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@@
   (junction (at 69.85 123.19) (diameter 0) (color 0 0 0 0)
   )
+  (no_connect (at 363.982 169.418))
   (no_connect (at 49.53 71.12))
   (no_connect (at 199.644 220.726))
-  (no_connect (at 363.982 187.198))
-  (no_connect (at 363.982 166.878))
   (no_connect (at 363.982 184.658))
   (no_connect (at 276.098 179.832))
+  (no_connect (at 329.184 240.538))
   (no_connect (at 310.642 192.532))
   (no_connect (at 115.57 64.77))
-  (no_connect (at 363.982 182.118))
   (no_connect (at 156.21 82.55))
   (no_connect (at 156.21 54.61))
-  (no_connect (at 363.982 177.038))
   (no_connect (at 115.57 69.85))
   (no_connect (at 156.21 59.69))
@@
   (no_connect (at 346.71 138.43))
   (no_connect (at 194.564 208.026))
+  (no_connect (at 363.982 199.898))
   (no_connect (at 199.644 177.546))
   (no_connect (at 363.982 197.358))
@@
   (no_connect (at 115.57 74.93))
   (no_connect (at 156.21 77.47))
+  (no_connect (at 363.982 174.498))
   (no_connect (at 310.642 197.612))
   (no_connect (at 156.21 80.01))
+  (no_connect (at 363.982 194.818))
   (no_connect (at 156.21 57.15))
-  (no_connect (at 363.982 171.958))
   (no_connect (at 156.21 52.07))
   (no_connect (at 199.644 197.866))
-  (no_connect (at 363.982 192.278))
+  (no_connect (at 363.982 179.578))
   (no_connect (at 156.21 64.77))
   (no_connect (at 194.564 185.166))
@@
     (stroke (width 0) (type default))
   )
-  (wire (pts (xy 329.438 230.378) (xy 335.28 230.378))
-    (stroke (width 0) (type default))
-  )
   (wire (pts (xy 77.47 123.19) (xy 85.09 123.19))
     (stroke (width 0) (type default))
@@
     (stroke (width 0) (type default))
   )
+  (wire (pts (xy 329.438 230.378) (xy 335.28 230.378))
+    (stroke (width 0) (type default))
+  )
   (wire (pts (xy 228.6 126.492) (xy 228.6 127.762))
     (stroke (width 0) (type default))
@@
     (stroke (width 0) (type default))
   )
-  (wire (pts (xy 325.882 237.998) (xy 335.28 237.998))
-    (stroke (width 0) (type default))
-  )
   (wire (pts (xy 329.438 217.678) (xy 335.28 217.678))
     (stroke (width 0) (type default))
@@
     (stroke (width 0) (type default))
   )
-  (wire (pts (xy 325.882 232.918) (xy 335.28 232.918))
+  (wire (pts (xy 329.438 232.918) (xy 335.28 232.918))
     (stroke (width 0) (type default))
   )
@@
     (stroke (width 0) (type default))
   )
+  (wire (pts (xy 329.184 237.998) (xy 335.28 237.998))
+    (stroke (width 0) (type default))
+  )
   (wire (pts (xy 130.81 254) (xy 143.51 254))
     (stroke (width 0) (type default))
@@
     (effects (font (size 1.27 1.27)) (justify left bottom))
   )
-  (label "PE9" (at 329.438 230.378 0) (fields_autoplaced)
-    (effects (font (size 1.27 1.27)) (justify left bottom))
-  )
   (label "PD0" (at 276.098 187.452 0) (fields_autoplaced)
     (effects (font (size 1.27 1.27)) (justify left bottom))
@@
     (effects (font (size 1.27 1.27)) (justify left bottom))
   )
-  (label "CAN-" (at 325.882 232.918 0) (fields_autoplaced)
-    (effects (font (size 1.27 1.27)) (justify left bottom))
-  )
   (label "PE1" (at 79.248 167.64 0) (fields_autoplaced)
     (effects (font (size 1.27 1.27)) (justify left bottom))
@@
     (effects (font (size 1.27 1.27)) (justify left bottom))
   )
-  (label "PE12" (at 359.664 169.418 0) (fields_autoplaced)
-    (effects (font (size 1.27 1.27)) (justify left bottom))
-  )
   (label "PE6" (at 329.438 207.518 0) (fields_autoplaced)
     (effects (font (size 1.27 1.27)) (justify left bottom))
@@
     (effects (font (size 1.27 1.27)) (justify left bottom))
   )
+  (label "CAN-" (at 329.438 235.458 0) (fields_autoplaced)
+    (effects (font (size 1.27 1.27)) (justify left bottom))
+  )
   (label "PE0" (at 306.324 182.372 0) (fields_autoplaced)
     (effects (font (size 1.27 1.27)) (justify left bottom))
@@
     (effects (font (size 1.27 1.27)) (justify left bottom))
   )
-  (label "PE14" (at 359.156 179.578 0) (fields_autoplaced)
-    (effects (font (size 1.27 1.27)) (justify left bottom))
-  )
   (label "SWDIO" (at 133.35 175.26 0) (fields_autoplaced)
     (effects (font (size 1.27 1.27)) (justify left bottom))
@@
     (effects (font (size 1.27 1.27)) (justify left bottom))
   )
+  (label "PE11" (at 359.41 166.878 0) (fields_autoplaced)
+    (effects (font (size 1.27 1.27)) (justify left bottom))
+  )
   (label "PC4" (at 329.438 194.818 0) (fields_autoplaced)
     (effects (font (size 1.27 1.27)) (justify left bottom))
@@
     (effects (font (size 1.27 1.27)) (justify left bottom))
   )
-  (label "CAN+" (at 325.882 237.998 0) (fields_autoplaced)
-    (effects (font (size 1.27 1.27)) (justify left bottom))
-  )
   (label "PD7" (at 276.098 223.012 0) (fields_autoplaced)
     (effects (font (size 1.27 1.27)) (justify left bottom))
@@
     (effects (font (size 1.27 1.27)) (justify left bottom))
   )
+  (label "PE14" (at 359.41 182.118 0) (fields_autoplaced)
+    (effects (font (size 1.27 1.27)) (justify left bottom))
+  )
   (label "GP_LED" (at 329.438 222.758 0) (fields_autoplaced)
     (effects (font (size 1.27 1.27)) (justify left bottom))
@@
     (effects (font (size 1.27 1.27)) (justify left bottom))
   )
-  (label "PE11" (at 329.184 240.538 0) (fields_autoplaced)
-    (effects (font (size 1.27 1.27)) (justify left bottom))
-  )
   (label "PC1" (at 133.604 228.6 0) (fields_autoplaced)
     (effects (font (size 1.27 1.27)) (justify left bottom))
@@
     (effects (font (size 1.27 1.27)) (justify left bottom))
   )
+  (label "PB10" (at 359.41 192.278 0) (fields_autoplaced)
+    (effects (font (size 1.27 1.27)) (justify left bottom))
+  )
   (label "PB13" (at 133.604 215.9 0) (fields_autoplaced)
     (effects (font (size 1.27 1.27)) (justify left bottom))
@@
     (effects (font (size 1.27 1.27)) (justify left bottom))
   )
+  (label "PE15" (at 359.41 187.198 0) (fields_autoplaced)
+    (effects (font (size 1.27 1.27)) (justify left bottom))
+  )
   (label "PA8" (at 306.324 179.832 0) (fields_autoplaced)
     (effects (font (size 1.27 1.27)) (justify left bottom))
@@
     (effects (font (size 1.27 1.27)) (justify left bottom))
   )
-  (label "PB13" (at 276.098 174.752 0) (fields_autoplaced)
+  (label "CAN+" (at 329.438 230.378 0) (fields_autoplaced)
     (effects (font (size 1.27 1.27)) (justify left bottom))
   )
-  (label "USB_D+" (at 107.95 54.61 0) (fields_autoplaced)
+  (label "PB13" (at 276.098 174.752 0) (fields_autoplaced)
     (effects (font (size 1.27 1.27)) (justify left bottom))
   )
-  (label "PE13" (at 359.156 174.498 0) (fields_autoplaced)
+  (label "USB_D+" (at 107.95 54.61 0) (fields_autoplaced)
     (effects (font (size 1.27 1.27)) (justify left bottom))
   )
@@
     (effects (font (size 1.27 1.27)) (justify left bottom))
   )
+  (label "PE10" (at 329.184 237.998 0) (fields_autoplaced)
+    (effects (font (size 1.27 1.27)) (justify left bottom))
+  )
   (label "PD3" (at 79.248 215.9 0) (fields_autoplaced)
     (effects (font (size 1.27 1.27)) (justify left bottom))
@@
     (effects (font (size 1.27 1.27)) (justify left bottom))
   )
-  (label "PE15" (at 358.902 194.818 0) (fields_autoplaced)
-    (effects (font (size 1.27 1.27)) (justify left bottom))
-  )
   (label "NRST" (at 78.74 142.24 0) (fields_autoplaced)
     (effects (font (size 1.27 1.27)) (justify left bottom))
@@
     (effects (font (size 1.27 1.27)) (justify right bottom))
   )
+  (label "PE12" (at 359.41 171.958 0) (fields_autoplaced)
+    (effects (font (size 1.27 1.27)) (justify left bottom))
+  )
   (label "SWO" (at 280.67 78.74 0) (fields_autoplaced)
     (effects (font (size 1.27 1.27)) (justify left bottom))
@@
     (effects (font (size 1.27 1.27)) (justify left bottom))
   )
-  (label "PB10" (at 359.156 199.898 0) (fields_autoplaced)
-    (effects (font (size 1.27 1.27)) (justify left bottom))
-  )
   (label "PB9" (at 133.604 208.28 0) (fields_autoplaced)
     (effects (font (size 1.27 1.27)) (justify left bottom))
@@
     (effects (font (size 1.27 1.27)) (justify left bottom))
   )
-  (label "PE10" (at 329.438 235.458 0) (fields_autoplaced)
-    (effects (font (size 1.27 1.27)) (justify left bottom))
-  )
   (label "PB4" (at 276.098 228.092 0) (fields_autoplaced)
     (effects (font (size 1.27 1.27)) (justify left bottom))
@@
     (effects (font (size 1.27 1.27)) (justify left bottom))
   )
+  (label "PE13" (at 359.41 177.038 0) (fields_autoplaced)
+    (effects (font (size 1.27 1.27)) (justify left bottom))
+  )
   (label "PA1" (at 134.112 144.78 0) (fields_autoplaced)
     (effects (font (size 1.27 1.27)) (justify left bottom))
@@
     (effects (font (size 1.27 1.27)) (justify left bottom))
   )
+  (label "PE9" (at 329.438 232.918 0) (fields_autoplaced)
+    (effects (font (size 1.27 1.27)) (justify left bottom))
+  )
   (label "PE0" (at 79.248 165.1 0) (fields_autoplaced)
     (effects (font (size 1.27 1.27)) (justify left bottom))
@@
       (effects (font (size 1.27 1.27)) hide)
     )
-    (property "JLCPCB" "" (at 307.34 68.58 0)
+    (property "JLCPCB" "C5504987" (at 307.34 68.58 0)
       (effects (font (size 1.27 1.27)) hide)
     )
@@
       (effects (font (size 1.27 1.27)) hide)
     )
-    (property "JLCPCB" "" (at 34.29 58.42 0)
+    (property "JLCPCB" "C3020560" (at 34.29 58.42 0)
       (effects (font (size 1.27 1.27)) hide)
     )
@@
       (effects (font (size 1.27 1.27)) hide)
     )
-    (property "JLCPCB" "" (at 107.95 205.74 0)
+    (property "JLCPCB" "C91929" (at 107.95 205.74 0)
       (effects (font (size 1.27 1.27)) hide)
     )
@@
       (effects (font (size 1.27 1.27)))
     )
-    (property "Footprint" "Capacitor_SMD:C_0603_1608Metric_Pad1.08x0.95mm_HandSolder" (at 43.18 201.422 90)
+    (property "Footprint" "Resistor_SMD:R_0603_1608Metric_Pad0.98x0.95mm_HandSolder" (at 43.18 201.422 90)
       (effects (font (size 1.27 1.27)) hide)
     )

Commit message: send for fab
Parts:
- X1: JLCPCB (none) -> C6106563
Changed lines of the file:
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@@
       (effects (font (size 1.27 1.27)) hide)
     )
-    (property "JLCPCB" "" (at 30.48 203.2 0)
+    (property "JLCPCB" "C6106563" (at 30.48 203.2 0)
       (effects (font (size 1.27 1.27)) hide)
     )
